Commit message: lift block env

File: urdf/box.urdf (robot description, URDF)
Before this commit: robot box, 1 links, 0 joints
Links:
- link box: geometry collision box size=0.03 0.03 0.02; visual box size=0.03 0.03 0.02

Commit message: slim

File: urdf/box.urdf (robot description, URDF)
Before this commit: robot box, 1 links, 0 joints
Links:
- link box: geometry collision box size=0.08 0.08 0.02; visual box size=0.08 0.08 0.02

Commit message: naive re-orientation

File: urdf/box.urdf (robot description, URDF)
Before this commit: robot box, 1 links, 0 joints
Links:
- link box: geometry collision box size=0.05 0.05 0.02; visual box size=0.05 0.05 0.02

Commit message: vectask env + PPO + fixed object + fixed start & goal position

File: urdf/box.urdf (robot description, URDF)
Before this commit: robot box, 1 links, 0 joints
Links:
- link box: geometry collision box size=0.04 0.04 0.04; visual box size=0.04 0.04 0.04

File: urdf/tablebot_row_16.urdf (robot description, URDF)
Before this commit: robot tablebot, 49 links, 48 joints
Links:
- removed link cylinder_0_0
- removed link cylinder_0_1
- removed link cylinder_0_10
- removed link cylinder_0_11
- removed link cylinder_0_12
- removed link cylinder_0_13
- removed link cylinder_0_14
- removed link cylinder_0_15
- removed link cylinder_0_2
- removed link cylinder_0_3
- removed link cylinder_0_4
- removed link cylinder_0_5
- removed link cylinder_0_6
- removed link cylinder_0_7
- removed link cylinder_0_8
- removed link cylinder_0_9
- removed link link_0_0
- removed link link_0_1
- removed link link_0_10
- removed link link_0_11
- removed link link_0_12
- removed link link_0_13
- removed link link_0_14
- removed link link_0_15
- removed link link_0_2
- removed link link_0_3
- removed link link_0_4
- removed link link_0_5
- removed link link_0_6
- removed link link_0_7
- removed link link_0_8
- removed link link_0_9
- removed link sphere_0_0
- removed link sphere_0_1
- removed link sphere_0_10
- removed link sphere_0_11
- removed link sphere_0_12
- removed link sphere_0_13
- removed link sphere_0_14
- removed link sphere_0_15
- removed link sphere_0_2
- removed link sphere_0_3
- removed link sphere_0_4
- removed link sphere_0_5
- removed link sphere_0_6
- removed link sphere_0_7
- removed link sphere_0_8
- removed link sphere_0_9
- added link cylinder_10_10, mass 0.05; collision cylinder length=0.01 radius=0.009; visual cylinder length=0.01 radius=0.009
- added link cylinder_10_11, mass 0.05; collision cylinder length=0.01 radius=0.009; visual cylinder length=0.01 radius=0.009
- added link cylinder_10_12, mass 0.05; collision cylinder length=0.01 radius=0.009; visual cylinder length=0.01 radius=0.009
- added link cylinder_10_13, mass 0.05; collision cylinder length=0.01 radius=0.009; visual cylinder length=0.01 radius=0.009
- added link cylinder_10_14, mass 0.05; collision cylinder length=0.01 radius=0.009; visual cylinder length=0.01 radius=0.009
- added link cylinder_10_15, mass 0.05; collision cylinder length=0.01 radius=0.009; visual cylinder length=0.01 radius=0.009
- added link cylinder_10_16, mass 0.05; collision cylinder length=0.01 radius=0.009; visual cylinder length=0.01 radius=0.009
- added link cylinder_10_17, mass 0.05; collision cylinder length=0.01 radius=0.009; visual cylinder length=0.01 radius=0.009
- added link cylinder_10_18, mass 0.05; collision cylinder length=0.01 radius=0.009; visual cylinder length=0.01 radius=0.009
- added link cylinder_10_19, mass 0.05; collision cylinder length=0.01 radius=0.009; visual cylinder length=0.01 radius=0.009
- added link cylinder_10_20, mass 0.05; collision cylinder length=0.01 radius=0.009; visual cylinder length=0.01 radius=0.009
- added link cylinder_10_21, mass 0.05; collision cylinder length=0.01 radius=0.009; visual cylinder length=0.01 radius=0.009
- added link cylinder_10_22, mass 0.05; collision cylinder length=0.01 radius=0.009; visual cylinder length=0.01 radius=0.009
- added link cylinder_10_23, mass 0.05; collision cylinder length=0.01 radius=0.009; visual cylinder length=0.01 radius=0.009
- added link cylinder_10_24, mass 0.05; collision cylinder length=0.01 radius=0.009; visual cylinder length=0.01 radius=0.009
- added link cylinder_10_25, mass 0.05; collision cylinder length=0.01 radius=0.009; visual cylinder length=0.01 radius=0.009
- added link link_10_10, mass 0.5; collision box size=0.016 0.016 0.055; visual box size=0.016 0.016 0.055
- added link link_10_11, mass 0.5; collision box size=0.016 0.016 0.055; visual box size=0.016 0.016 0.055
- added link link_10_12, mass 0.5; collision box size=0.016 0.016 0.055; visual box size=0.016 0.016 0.055
- added link link_10_13, mass 0.5; collision box size=0.016 0.016 0.055; visual box size=0.016 0.016 0.055
- added link link_10_14, mass 0.5; collision box size=0.016 0.016 0.055; visual box size=0.016 0.016 0.055
- added link link_10_15, mass 0.5; collision box size=0.016 0.016 0.055; visual box size=0.016 0.016 0.055
- added link link_10_16, mass 0.5; collision box size=0.016 0.016 0.055; visual box size=0.016 0.016 0.055
- added link link_10_17, mass 0.5; collision box size=0.016 0.016 0.055; visual box size=0.016 0.016 0.055
- added link link_10_18, mass 0.5; collision box size=0.016 0.016 0.055; visual box size=0.016 0.016 0.055
- added link link_10_19, mass 0.5; collision box size=0.016 0.016 0.055; visual box size=0.016 0.016 0.055
- added link link_10_20, mass 0.5; collision box size=0.016 0.016 0.055; visual box size=0.016 0.016 0.055
- added link link_10_21, mass 0.5; collision box size=0.016 0.016 0.055; visual box size=0.016 0.016 0.055
- added link link_10_22, mass 0.5; collision box size=0.016 0.016 0.055; visual box size=0.016 0.016 0.055
- added link link_10_23, mass 0.5; collision box size=0.016 0.016 0.055; visual box size=0.016 0.016 0.055
- added link link_10_24, mass 0.5; collision box size=0.016 0.016 0.055; visual box size=0.016 0.016 0.055
- added link link_10_25, mass 0.5; collision box size=0.016 0.016 0.055; visual box size=0.016 0.016 0.055
- added link sphere_10_10, mass 0.05; collision sphere radius=0.009; visual sphere radius=0.009
- added link sphere_10_11, mass 0.05; collision sphere radius=0.009; visual sphere radius=0.009
- added link sphere_10_12, mass 0.05; collision sphere radius=0.009; visual sphere radius=0.009
- added link sphere_10_13, mass 0.05; collision sphere radius=0.009; visual sphere radius=0.009
- added link sphere_10_14, mass 0.05; collision sphere radius=0.009; visual sphere radius=0.009
- added link sphere_10_15, mass 0.05; collision sphere radius=0.009; visual sphere radius=0.009
- added link sphere_10_16, mass 0.05; collision sphere radius=0.009; visual sphere radius=0.009
- added link sphere_10_17, mass 0.05; collision sphere radius=0.009; visual sphere radius=0.009
- added link sphere_10_18, mass 0.05; collision sphere radius=0.009; visual sphere radius=0.009
- added link sphere_10_19, mass 0.05; collision sphere radius=0.009; visual sphere radius=0.009
- added link sphere_10_20, mass 0.05; collision sphere radius=0.009; visual sphere radius=0.009
- added link sphere_10_21, mass 0.05; collision sphere radius=0.009; visual sphere radius=0.009
- added link sphere_10_22, mass 0.05; collision sphere radius=0.009; visual sphere radius=0.009
- added link sphere_10_23, mass 0.05; collision sphere radius=0.009; visual sphere radius=0.009
- added link sphere_10_24, mass 0.05; collision sphere radius=0.009; visual sphere radius=0.009
- added link sphere_10_25, mass 0.05; collision sphere radius=0.009; visual sphere radius=0.009
Joints:
- removed joint cylinder2base_0_0
- removed joint cylinder2base_0_1
- removed joint cylinder2base_0_10
- removed joint cylinder2base_0_11
- removed joint cylinder2base_0_12
- removed joint cylinder2base_0_13
- removed joint cylinder2base_0_14
- removed joint cylinder2base_0_15
- removed joint cylinder2base_0_2
- removed joint cylinder2base_0_3
- removed joint cylinder2base_0_4
- removed joint cylinder2base_0_5
- removed joint cylinder2base_0_6
- removed joint cylinder2base_0_7
- removed joint cylinder2base_0_8
- removed joint cylinder2base_0_9
- removed joint joint_0_0
- removed joint joint_0_1
- removed joint joint_0_10
- removed joint joint_0_11
- removed joint joint_0_12
- removed joint joint_0_13
- removed joint joint_0_14
- removed joint joint_0_15
- removed joint joint_0_2
- removed joint joint_0_3
- removed joint joint_0_4
- removed joint joint_0_5
- removed joint joint_0_6
- removed joint joint_0_7
- removed joint joint_0_8
- removed joint joint_0_9
- removed joint sphere2cylinder_0_0
- removed joint sphere2cylinder_0_1
- removed joint sphere2cylinder_0_10
- removed joint sphere2cylinder_0_11
- removed joint sphere2cylinder_0_12
- removed joint sphere2cylinder_0_13
- removed joint sphere2cylinder_0_14
- removed joint sphere2cylinder_0_15
- removed joint sphere2cylinder_0_2
- removed joint sphere2cylinder_0_3
- removed joint sphere2cylinder_0_4
- removed joint sphere2cylinder_0_5
- removed joint sphere2cylinder_0_6
- removed joint sphere2cylinder_0_7
- removed joint sphere2cylinder_0_8
- removed joint sphere2cylinder_0_9
- added joint cylinder2base_10_10: type fixed, parent link_10_10, child cylinder_10_10, origin xyz=0 0 0.01
- added joint cylinder2base_10_11: type fixed, parent link_10_11, child cylinder_10_11, origin xyz=0 0 0.01
- added joint cylinder2base_10_12: type fixed, parent link_10_12, child cylinder_10_12, origin xyz=0 0 0.01
- added joint cylinder2base_10_13: type fixed, parent link_10_13, child cylinder_10_13, origin xyz=0 0 0.01
- added joint cylinder2base_10_14: type fixed, parent link_10_14, child cylinder_10_14, origin xyz=0 0 0.01
- added joint cylinder2base_10_15: type fixed, parent link_10_15, child cylinder_10_15, origin xyz=0 0 0.01
- added joint cylinder2base_10_16: type fixed, parent link_10_16, child cylinder_10_16, origin xyz=0 0 0.01
- added joint cylinder2base_10_17: type fixed, parent link_10_17, child cylinder_10_17, origin xyz=0 0 0.01
- added joint cylinder2base_10_18: type fixed, parent link_10_18, child cylinder_10_18, origin xyz=0 0 0.01
- added joint cylinder2base_10_19: type fixed, parent link_10_19, child cylinder_10_19, origin xyz=0 0 0.01
- added joint cylinder2base_10_20: type fixed, parent link_10_20, child cylinder_10_20, origin xyz=0 0 0.01
- added joint cylinder2base_10_21: type fixed, parent link_10_21, child cylinder_10_21, origin xyz=0 0 0.01
- added joint cylinder2base_10_22: type fixed, parent link_10_22, child cylinder_10_22, origin xyz=0 0 0.01
- added joint cylinder2base_10_23: type fixed, parent link_10_23, child cylinder_10_23, origin xyz=0 0 0.01
- added joint cylinder2base_10_24: type fixed, parent link_10_24, child cylinder_10_24, origin xyz=0 0 0.01
- added joint cylinder2base_10_25: type fixed, parent link_10_25, child cylinder_10_25, origin xyz=0 0 0.01
- added joint joint_10_10: type prismatic, parent table_base, child link_10_10, origin xyz=0.018000000000000002 0.018000000000000002 0, axis 0 0 1, limit lower=0 upper=0.045 effort=4 velocity=0.05
- added joint joint_10_11: type prismatic, parent table_base, child link_10_11, origin xyz=0.018000000000000002 0.038 0, axis 0 0 1, limit lower=0 upper=0.045 effort=4 velocity=0.05
- added joint joint_10_12: type prismatic, parent table_base, child link_10_12, origin xyz=0.018000000000000002 0.058 0, axis 0 0 1, limit lower=0 upper=0.045 effort=4 velocity=0.05
- added joint joint_10_13: type prismatic, parent table_base, child link_10_13, origin xyz=0.018000000000000002 0.078 0, axis 0 0 1, limit lower=0 upper=0.045 effort=4 velocity=0.05
- added joint joint_10_14: type prismatic, parent table_base, child link_10_14, origin xyz=0.018000000000000002 0.098 0, axis 0 0 1, limit lower=0 upper=0.045 effort=4 velocity=0.05
- added joint joint_10_15: type prismatic, parent table_base, child link_10_15, origin xyz=0.018000000000000002 0.118 0, axis 0 0 1, limit lower=0 upper=0.045 effort=4 velocity=0.05
- added joint joint_10_16: type prismatic, parent table_base, child link_10_16, origin xyz=0.018000000000000002 0.138 0, axis 0 0 1, limit lower=0 upper=0.045 effort=4 velocity=0.05
- added joint joint_10_17: type prismatic, parent table_base, child link_10_17, origin xyz=0.018000000000000002 0.158 0, axis 0 0 1, limit lower=0 upper=0.045 effort=4 velocity=0.05
- added joint joint_10_18: type prismatic, parent table_base, child link_10_18, origin xyz=0.018000000000000002 0.17800000000000002 0, axis 0 0 1, limit lower=0 upper=0.045 effort=4 velocity=0.05
- added joint joint_10_19: type prismatic, parent table_base, child link_10_19, origin xyz=0.018000000000000002 0.198 0, axis 0 0 1, limit lower=0 upper=0.045 effort=4 velocity=0.05
- added joint joint_10_20: type prismatic, parent table_base, child link_10_20, origin xyz=0.018000000000000002 0.21800000000000003 0, axis 0 0 1, limit lower=0 upper=0.045 effort=4 velocity=0.05
- added joint joint_10_21: type prismatic, parent table_base, child link_10_21, origin xyz=0.018000000000000002 0.238 0, axis 0 0 1, limit lower=0 upper=0.045 effort=4 velocity=0.05
- added joint joint_10_22: type prismatic, parent table_base, child link_10_22, origin xyz=0.018000000000000002 0.258 0, axis 0 0 1, limit lower=0 upper=0.045 effort=4 velocity=0.05
- added joint joint_10_23: type prismatic, parent table_base, child link_10_23, origin xyz=0.018000000000000002 0.278 0, axis 0 0 1, limit lower=0 upper=0.045 effort=4 velocity=0.05
- added joint joint_10_24: type prismatic, parent table_base, child link_10_24, origin xyz=0.018000000000000002 0.29800000000000004 0, axis 0 0 1, limit lower=0 upper=0.045 effort=4 velocity=0.05
- added joint joint_10_25: type prismatic, parent table_base, child link_10_25, origin xyz=0.018000000000000002 0.318 0, axis 0 0 1, limit lower=0 upper=0.045 effort=4 velocity=0.05
- added joint sphere2cylinder_10_10: type fixed, parent cylinder_10_10, child sphere_10_10, origin xyz=0 0 0
- added joint sphere2cylinder_10_11: type fixed, parent cylinder_10_11, child sphere_10_11, origin xyz=0 0 0
- added joint sphere2cylinder_10_12: type fixed, parent cylinder_10_12, child sphere_10_12, origin xyz=0 0 0
- added joint sphere2cylinder_10_13: type fixed, parent cylinder_10_13, child sphere_10_13, origin xyz=0 0 0
- added joint sphere2cylinder_10_14: type fixed, parent cylinder_10_14, child sphere_10_14, origin xyz=0 0 0
- added joint sphere2cylinder_10_15: type fixed, parent cylinder_10_15, child sphere_10_15, origin xyz=0 0 0
- added joint sphere2cylinder_10_16: type fixed, parent cylinder_10_16, child sphere_10_16, origin xyz=0 0 0
- added joint sphere2cylinder_10_17: type fixed, parent cylinder_10_17, child sphere_10_17, origin xyz=0 0 0
- added joint sphere2cylinder_10_18: type fixed, parent cylinder_10_18, child sphere_10_18, origin xyz=0 0 0
- added joint sphere2cylinder_10_19: type fixed, parent cylinder_10_19, child sphere_10_19, origin xyz=0 0 0
- added joint sphere2cylinder_10_20: type fixed, parent cylinder_10_20, child sphere_10_20, origin xyz=0 0 0
- added joint sphere2cylinder_10_21: type fixed, parent cylinder_10_21, child sphere_10_21, origin xyz=0 0 0
- added joint sphere2cylinder_10_22: type fixed, parent cylinder_10_22, child sphere_10_22, origin xyz=0 0 0
- added joint sphere2cylinder_10_23: type fixed, parent cylinder_10_23, child sphere_10_23, origin xyz=0 0 0
- added joint sphere2cylinder_10_24: type fixed, parent cylinder_10_24, child sphere_10_24, origin xyz=0 0 0
- added joint sphere2cylinder_10_25: type fixed, parent cylinder_10_25, child sphere_10_25, origin xyz=0 0 0
